Commit message: To test

File: src/my_robot/urdf/my_robot.xacro (robot description, xacro)
@@ -148,4 +148,6 @@
       </visual>
   </link>
+  <link name="camera_link_optical">
+  </link>
   <joint type="continuous" name="left_wheel_hinge">
     <origin xyz="0 0.15 0" rpy="0 0 0"/>
@@ -176,4 +178,9 @@
     <axis xyz="0 1 0" rpy="0 0 0"/>
   </joint>
+  <joint name="camera_optical_joint" type="fixed">
+    <origin xyz="0 0 0" rpy="-1.5707 0 -1.5707"/>
+    <parent link="camera"/>
+    <child link="camera_link_optical"/>
+  </joint>
   <gazebo reference="left_wheel">
       <material>Gazebo/Green</material>
